File: biosensorbox/biosensorbox.kicad_pcb (KiCad board)
At the start: 2 copper layers, 60 x 40 mm, 54 parts, among them J1 USB_B_Mini, J2 Display, Q1 MDD2302, Q2 MDD2302, SW1 BootButton, SW2 ResetButton, SW3 DisplayButton, U1 ESP32-S3-WROOM-1, U2 AMS1117-3.3, U3 SRV05-4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

Commit message: Finished layout and generated gerbers ! PCB is done !
Parts:
- added G***: LOGO, LOGO, B.Cu at (127.0, 93.3)
- added G***: LOGO, LOGO, B.Cu at (148.6, 98.0)
- D1, D2, D3, D4, D6, D7, D8, D9: footprint LED_SMD:LED_0603_1608Metric -> LED_SMD:LED_0805_2012Metric
- moved J2 12.6 mm to (111.6, 94.0), turned to 0 degrees
- moved R13 1.74 mm to (153.0, 83.9)
- moved R12 1.74 mm to (156.2, 83.9)
- moved C11 1.46 mm to (158.3, 85.5)
- moved C14 1.00 mm to (152.1, 90.9), turned to 180 degrees
- moved C12 0.68 mm to (154.9, 91.7)
- moved U5 0.64 mm to (154.1, 87.4)
- moved R5 0.64 mm to (140.4, 75.6), turned to 90 degrees
- moved SW1 0.57 mm to (158.7, 94.5)
- moved C13 0.55 mm to (157.6, 87.8), turned to 90 degrees
- moved Q2 0.55 mm to (133.6, 67.9)
- moved R16 0.54 mm to (127.9, 80.9)
- moved R7 0.53 mm to (126.2, 75.7)
- moved R6 0.48 mm to (133.1, 80.9)
- moved R4 0.47 mm to (133.3, 70.4)
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Connections:
- J1 pad 6: unconnected-(J1-Shield-Pad6) -> GND
Routing:
- net +3V3: track 45.8 -> 190.9 mm, vias 0 -> 5
- net GND: track 0.00 -> 140.9 mm, vias 0 -> 36
- net /SCL_DISP: track 0.00 -> 65.1 mm, vias 0 -> 2
- net /SDA_DISP: track 0.00 -> 63.6 mm, vias 0 -> 2
- net Net-(U1-EN): track 2.18 -> 46.7 mm, vias 0 -> 2
- net Net-(Q1-D): track 0.00 -> 39.8 mm
- net Net-(Q2-D): track 0.00 -> 32.3 mm
- net /DisplayButton: track 10.7 -> 28.5 mm, vias 0 -> 2
- net /INT_IMU: track 0.00 -> 16.6 mm, vias 0 -> 2
- net Net-(Q1-G): track 0.00 -> 14.5 mm, vias 0 -> 2
- net Net-(Q2-G): track 0.00 -> 12.3 mm
- net /D+: track 3.63 -> 15.2 mm
- net /D-: track 3.18 -> 14.6 mm
- net VBUS: track 7.77 -> 17.8 mm
- net /SCL_IMU: track 0.00 -> 5.83 mm
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- added copper zone on In1.Cu, net GND
- added copper zone on In2.Cu, net GND
Other:
- board size 60 x 40 mm -> 52.6 x 40 mm
- copper layers 2 -> 4
- board text added: "+"
- board text added: "Bio-Watch Project V1 by Jad Haidamous"
